Commit message: feat: Add open01_description ROS2 package with URDF model
- Added open01.urdf defining robot structure with base_link, wheels, IMU, and TOF sensor links.
- Migrated package from ROS1 catkin to ROS2 ament_cmake build system.
- Updated CMakeLists.txt and package.xml for ROS2 compatibility.
- Renamed all Robot_Assembly_1 references to open01_description.
- Added joint_names_open01.yaml for joint configuration.
- Updated .gitignore to exclude ROS2 build artifacts.

File: robot_ros2/ros2_ws/src/open01_description/urdf/open01.urdf (robot description, URDF)
Before this commit: robot Robot_Assembly_1, 7 links, 6 joints
Links:
- link IMU: geometry collision mesh filename=package://open01_description/meshes/IMU.STL; visual mesh filename=package://open01_description/meshes/IMU.STL
- link Left_Wheel: geometry collision mesh filename=package://open01_description/meshes/Left_Wheel.STL; visual mesh filename=package://open01_description/meshes/Left_Wheel.STL
- link Right_Wheel: geometry collision mesh filename=package://open01_description/meshes/Right_Wheel.STL; visual mesh filename=package://open01_description/meshes/Right_Wheel.STL
- link TOF_Back: geometry collision mesh filename=package://open01_description/meshes/TOF_Back.STL; visual mesh filename=package://open01_description/meshes/TOF_Back.STL
- link TOF_Left: geometry collision mesh filename=package://open01_description/meshes/TOF_Left.STL; visual mesh filename=package://open01_description/meshes/TOF_Left.STL
- link TOF_Right: geometry collision mesh filename=package://open01_description/meshes/TOF_Right.STL; visual mesh filename=package://open01_description/meshes/TOF_Right.STL
- link base_link: geometry collision mesh filename=package://open01_description/meshes/base_link.STL; visual mesh filename=package://open01_description/meshes/base_link.STL

Commit message: fix: Remove empty IMU mesh, lowercase STL extensions in URDF

File: robot_ros2/ros2_ws/src/open01_description/urdf/open01.urdf (robot description, URDF)
Before this commit: robot open01_description, 7 links, 6 joints
Links:
- link IMU: geometry 
- link Left_Wheel: geometry collision mesh filename=package://open01_description/meshes/Left_Wheel.stl; visual mesh filename=package://open01_description/meshes/Left_Wheel.stl
- link Right_Wheel: geometry collision mesh filename=package://open01_description/meshes/Right_Wheel.stl; visual mesh filename=package://open01_description/meshes/Right_Wheel.stl
- link TOF_Back: geometry collision mesh filename=package://open01_description/meshes/TOF_Back.stl; visual mesh filename=package://open01_description/meshes/TOF_Back.stl
- link TOF_Left: geometry collision mesh filename=package://open01_description/meshes/TOF_Left.stl; visual mesh filename=package://open01_description/meshes/TOF_Left.stl
- link TOF_Right: geometry collision mesh filename=package://open01_description/meshes/TOF_Right.stl; visual mesh filename=package://open01_description/meshes/TOF_Right.stl
- link base_link: geometry collision mesh filename=package://open01_description/meshes/base_link.stl; visual mesh filename=package://open01_description/meshes/base_link.stl
